File: stm32/stm32l432/projects/project04_ssd_1306_driver_demo/circuit/circuit.kicad_sch (KiCad schematic)
At the start: 4 parts, among them J1 HT16K33 Led Matrix, SW1 Right Btn, SW2 Left Btn, U1 STM32L432KCUx

Commit message: Updated documentation
Parts:
- removed J1: HT16K33 Led Matrix, symbol Connector_Generic:Conn_01x04
- added J?: SSD 1306, symbol Connector_Generic:Conn_01x04
Connections:
- net +5V: now also J?.2 (Pin_2)
- net GND: now also J?.1 (Pin_1)
- net at U1.20 (PA10): now also J?.4 (Pin_4)
- net at U1.19 (PA9): now also J?.3 (Pin_3)
Other:
- note added: "Project04 SSD 1306 Driver Demo"
- note removed: "Project03 HT16K33 Scroll text demo"
Changed lines of the file:
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@@
 	(generator_version "9.0")
 	(paper "A4")
-	(text "Project03 HT16K33 Scroll text demo"
+	(text "Project04 SSD 1306 Driver Demo"
 		(exclude_from_sim no)
 		(at 152.4 22.86 0)
@@
 	(wire
 		(pts
-			(xy 181.61 69.85) (xy 181.61 60.96)
-		)
-		(stroke
-			(width 0)
-			(type default)
-		)
-	)
-	(wire
-		(pts
 			(xy 133.35 63.5) (xy 133.35 66.04)
 		)
@@
 	(wire
 		(pts
+			(xy 181.61 63.5) (xy 181.61 69.85)
+		)
+		(stroke
+			(width 0)
+			(type default)
+		)
+	)
+	(wire
+		(pts
 			(xy 127 48.26) (xy 138.43 48.26)
 		)
@@
 	(wire
 		(pts
+			(xy 184.15 60.96) (xy 184.15 69.85)
+		)
+		(stroke
+			(width 0)
+			(type default)
+		)
+	)
+	(wire
+		(pts
 			(xy 127 63.5) (xy 133.35 63.5)
 		)
@@
 	(wire
 		(pts
-			(xy 191.77 67.31) (xy 191.77 44.45)
+			(xy 186.69 69.85) (xy 186.69 45.72)
 		)
 		(stroke
@@
 	(wire
 		(pts
-			(xy 194.31 69.85) (xy 194.31 45.72)
-		)
-		(stroke
-			(width 0)
-			(type default)
-		)
-	)
-	(wire
-		(pts
-			(xy 186.69 67.31) (xy 191.77 67.31)
-		)
-		(stroke
-			(width 0)
-			(type default)
-		)
-	)
-	(wire
-		(pts
 			(xy 138.43 63.5) (xy 140.97 63.5)
 		)
@@
 	(wire
 		(pts
-			(xy 191.77 44.45) (xy 186.69 44.45)
-		)
-		(stroke
-			(width 0)
-			(type default)
-		)
-	)
-	(wire
-		(pts
 			(xy 138.43 48.26) (xy 138.43 63.5)
 		)
@@
 	(wire
 		(pts
-			(xy 184.15 63.5) (xy 166.37 63.5)
+			(xy 189.23 45.72) (xy 196.85 45.72)
 		)
 		(stroke
@@
 	(wire
 		(pts
+			(xy 166.37 63.5) (xy 181.61 63.5)
+		)
+		(stroke
+			(width 0)
+			(type default)
+		)
+	)
+	(wire
+		(pts
 			(xy 116.84 63.5) (xy 114.3 63.5)
 		)
@@
 	(wire
 		(pts
-			(xy 189.23 69.85) (xy 194.31 69.85)
-		)
-		(stroke
-			(width 0)
-			(type default)
-		)
-	)
-	(wire
-		(pts
-			(xy 184.15 69.85) (xy 184.15 63.5)
+			(xy 166.37 60.96) (xy 184.15 60.96)
+		)
+		(stroke
+			(width 0)
+			(type default)
+		)
+	)
+	(wire
+		(pts
+			(xy 189.23 69.85) (xy 189.23 45.72)
 		)
 		(stroke
@@
 		(pts
 			(xy 107.95 48.26) (xy 107.95 53.34)
-		)
-		(stroke
-			(width 0)
-			(type default)
-		)
-	)
-	(wire
-		(pts
-			(xy 181.61 60.96) (xy 166.37 60.96)
-		)
-		(stroke
-			(width 0)
-			(type default)
-		)
-	)
-	(wire
-		(pts
-			(xy 186.69 69.85) (xy 186.69 67.31)
 		)
 		(stroke
@@
 	(symbol
 		(lib_id "power:+5V")
-		(at 194.31 45.72 0)
+		(at 186.69 45.72 0)
 		(unit 1)
 		(exclude_from_sim no)
@@
 		(fields_autoplaced yes)
 		(property "Reference" "#PWR02"
-			(at 194.31 49.53 0)
+			(at 186.69 49.53 0)
 			(effects
 				(font
@@
 		)
 		(property "Value" "+5V"
-			(at 194.31 40.64 0)
+			(at 186.69 40.64 0)
 			(effects
 				(font
@@
 		)
 		(property "Footprint" ""
-			(at 194.31 45.72 0)
+			(at 186.69 45.72 0)
 			(effects
 				(font
@@
 		)
 		(property "Datasheet" ""
-			(at 194.31 45.72 0)
+			(at 186.69 45.72 0)
 			(effects
 				(font
@@
 		)
 		(property "Description" "Power symbol creates a global label with name \"+5V\""
-			(at 194.31 45.72 0)
+			(at 186.69 45.72 0)
 			(effects
 				(font
@@
 	)
 	(symbol
-		(lib_id "Connector_Generic:Conn_01x04")
-		(at 186.69 74.93 270)
-		(unit 1)
-		(exclude_from_sim no)
-		(in_bom yes)
-		(on_board yes)
-		(dnp no)
-		(fields_autoplaced yes)
-		(property "Reference" "J1"
-			(at 185.42 78.74 90)
-			(effects
-				(font
-					(size 1.27 1.27)
-				)
-				(hide yes)
-			)
-		)
-		(property "Value" "HT16K33 Led Matrix"
-			(at 185.42 81.28 90)
-			(effects
-				(font
-					(size 1.27 1.27)
-				)
-			)
-		)
-		(property "Footprint" ""
-			(at 186.69 74.93 0)
-			(effects
-				(font
-					(size 1.27 1.27)
-				)
-				(hide yes)
-			)
-		)
-		(property "Datasheet" "~"
-			(at 186.69 74.93 0)
-			(effects
-				(font
-					(size 1.27 1.27)
-				)
-				(hide yes)
-			)
-		)
-		(property "Description" "Generic connector, single row, 01x04, script generated (kicad-library-utils/schlib/autogen/connector/)"
-			(at 186.69 74.93 0)
-			(effects
-				(font
-					(size 1.27 1.27)
-				)
-				(hide yes)
-			)
-		)
-		(pin "3"
-		)
-		(pin "4"
-		)
-		(pin "2"
-		)
-		(pin "1"
-		)
-		(instances
-			(project "circuit"
-				(path "/08ce7381-92fb-4307-ae53-565418cecde2"
-					(reference "J1")
-					(unit 1)
-				)
-			)
-		)
-	)
-	(symbol
 		(lib_id "power:GND")
 		(at 107.95 53.34 0)
@@
 	)
 	(symbol
+		(lib_name "Conn_01x04_1")
+		(lib_id "Connector_Generic:Conn_01x04")
+		(at 186.69 74.93 270)
+		(unit 1)
+		(exclude_from_sim no)
+		(in_bom yes)
+		(on_board yes)
+		(dnp no)
+		(fields_autoplaced yes)
+		(property "Reference" "J?"
+			(at 185.42 78.74 90)
+			(effects
+				(font
+					(size 1.27 1.27)
+				)
+				(hide yes)
+			)
+		)
+		(property "Value" "SSD 1306"
+			(at 185.42 81.28 90)
+			(effects
+				(font
+					(size 1.27 1.27)
+				)
+			)
+		)
+		(property "Footprint" ""
+			(at 186.69 74.93 0)
+			(effects
+				(font
+					(size 1.27 1.27)
+				)
+				(hide yes)
+			)
+		)
+		(property "Datasheet" "~"
+			(at 186.69 74.93 0)
+			(effects
+				(font
+					(size 1.27 1.27)
+				)
+				(hide yes)
+			)
+		)
+		(property "Description" "Generic connector, single row, 01x04, script generated (kicad-library-utils/schlib/autogen/connector/)"
+			(at 186.69 74.93 0)
+			(effects
+				(font
+					(size 1.27 1.27)
+				)
+				(hide yes)
+			)
+		)
+		(pin "3"
+		)
+		(pin "4"
+		)
+		(pin "2"
+		)
+		(pin "1"
+		)
+		(instances
+			(project "circuit"
+				(path "/08ce7381-92fb-4307-ae53-565418cecde2"
+					(reference "J?")
+					(unit 1)
+				)
+			)
+		)
+	)
+	(symbol
 		(lib_id "power:GND")
-		(at 186.69 44.45 0)
+		(at 196.85 45.72 0)
 		(unit 1)
 		(exclude_from_sim no)
@@
 		(fields_autoplaced yes)
 		(property "Reference" "#PWR01"
-			(at 186.69 50.8 0)
+			(at 196.85 52.07 0)
 			(effects
 				(font
@@
 		)
 		(property "Value" "GND"
-			(at 186.69 49.53 0)
+			(at 196.85 50.8 0)
 			(effects
 				(font
@@
 		)
 		(property "Footprint" ""
-			(at 186.69 44.45 0)
+			(at 196.85 45.72 0)
 			(effects
 				(font
@@
 		)
 		(property "Datasheet" ""
-			(at 186.69 44.45 0)
+			(at 196.85 45.72 0)
 			(effects
 				(font
@@
 		)
 		(property "Description" "Power symbol creates a global label with name \"GND\" , ground"
-			(at 186.69 44.45 0)
-			(effects
-				(font
+			(at 196.85 45.72 0)
+			(effects
+				(font
